Commit message: Update camera properties in ranger_complete.urdf.xacro and change material color in piper_description_prefixed.xacro

File: src/ranger_description/urdf/piper_description_prefixed.xacro (robot description, xacro)
@@ -414,6 +414,6 @@
           <box size="0.04 0.04 0.025"/>
         </geometry>
-        <material name="d405_black">
-          <color rgba="0.1 0.1 0.1 1.0"/>
+        <material name="silver">
+          <color rgba="0.8 0.8 0.8 1.0"/>
         </material>
       </visual>

File: src/ranger_description/urdf/ranger_complete.urdf.xacro (robot description, xacro)
@@ -14,9 +14,9 @@
   <xacro:property name="arm_y" value="0.0"/>
   <xacro:property name="arm_z" value="0.0"/>
-  <xacro:property name="piper_camera_x" value="0.0"/>
+  <xacro:property name="piper_camera_x" value="-0.085"/>
   <xacro:property name="piper_camera_y" value="0.0"/>
   <xacro:property name="piper_camera_z" value="0.05"/>
   <xacro:property name="piper_camera_roll" value="0.0"/>
-  <xacro:property name="piper_camera_pitch" value="0.0"/>
+  <xacro:property name="piper_camera_pitch" value="0.5236"/>
   <xacro:property name="piper_camera_yaw" value="0.0"/>
   <xacro:property name="mesh_dir" value="$(arg mesh_dir)"/>

Commit message: Add optical frame and joint for PiPER wrist camera in URDF

File: src/ranger_description/urdf/piper_description_prefixed.xacro (robot description, xacro)
@@ -430,4 +430,11 @@
       <origin xyz="${camera_xyz}" rpy="${camera_roll} ${camera_pitch - 1.5708} ${camera_yaw}"/>
     </joint>
+    <!-- PiPER wrist camera optical frame -->
+    <link name="${prefix}camera_optical_frame"/>
+    <joint name="${prefix}camera_optical_joint" type="fixed">
+      <parent link="${prefix}camera_link"/>
+      <child link="${prefix}camera_optical_frame"/>
+      <origin xyz="0 0 0" rpy="${-M_PI/2} 0 ${-M_PI/2}"/>
+    </joint>
     <link
       name="${prefix}link7">
