Commit message: Enhance PiPER arm macros with camera parameters and update URDF files for improved integration

File: src/ranger_description/urdf/piper_arm_macro.xacro (robot description, xacro)
@@ -4,6 +4,6 @@
   <xacro:include filename="$(find ranger_description)/urdf/piper_description_prefixed.xacro" />
   <!-- Wrapper macro to mount the PiPER arm to an arbitrary parent link. -->
-  <xacro:macro name="piper_arm" params="parent_link xyz:='0 0 0' rpy:='0 0 0' prefix:='piper_'">
-    <xacro:piper_with_gripper prefix="${prefix}" />
+  <xacro:macro name="piper_arm" params="parent_link xyz:='0 0 0' rpy:='0 0 0' prefix:='piper_' camera_xyz:='0 0 0.05' camera_rpy:='0 0 0'">
+    <xacro:piper_with_gripper prefix="${prefix}" camera_xyz="${camera_xyz}" camera_rpy="${camera_rpy}" />
     <!--
       Mount PiPER's world link to the requested parent.

File: src/ranger_description/urdf/piper_description_prefixed.xacro (robot description, xacro)
@@ -14,5 +14,5 @@
     </transmission>
   </xacro:macro>
-  <xacro:macro name="piper_with_gripper" params="prefix:='piper_'">
+  <xacro:macro name="piper_with_gripper" params="prefix:='piper_' camera_xyz:='0 0 0.05' camera_rpy:='0 0 0'">
   <!-- world -->
     <link name="${prefix}world"/>
@@ -399,4 +399,34 @@
       <child
         link="${prefix}gripper_base" />
+    </joint>
+    <!-- PiPER wrist camera (RealSense D405) -->
+    <link name="${prefix}camera_link">
+      <inertial>
+        <origin xyz="0 0 0" rpy="0 0 0" />
+        <mass value="0.07" />
+        <inertia ixx="0.00001298" ixy="0.0" ixz="0.0"
+                 iyy="0.00001298" iyz="0.0"
+                 izz="0.00001867" />
+      </inertial>
+      <visual>
+        <origin xyz="0 0 0" rpy="0 0 0" />
+        <geometry>
+          <box size="0.04 0.04 0.025"/>
+        </geometry>
+        <material name="d405_black">
+          <color rgba="0.1 0.1 0.1 1.0"/>
+        </material>
+      </visual>
+      <collision>
+        <origin xyz="0 0 0" rpy="0 0 0" />
+        <geometry>
+          <box size="0.04 0.04 0.025"/>
+        </geometry>
+      </collision>
+    </link>
+    <joint name="${prefix}camera_mount_joint" type="fixed">
+      <parent link="${prefix}gripper_base"/>
+      <child link="${prefix}camera_link"/>
+      <origin xyz="${camera_xyz}" rpy="${camera_rpy}"/>
     </joint>
     <link

File: src/ranger_description/urdf/ranger_complete.urdf.xacro (robot description, xacro)
@@ -14,4 +14,10 @@
   <xacro:property name="arm_y" value="0.0"/>
   <xacro:property name="arm_z" value="0.0"/>
+  <xacro:property name="piper_camera_x" value="0.0"/>
+  <xacro:property name="piper_camera_y" value="0.0"/>
+  <xacro:property name="piper_camera_z" value="0.05"/>
+  <xacro:property name="piper_camera_roll" value="0.0"/>
+  <xacro:property name="piper_camera_pitch" value="0.0"/>
+  <xacro:property name="piper_camera_yaw" value="0.0"/>
   <xacro:property name="mesh_dir" value="$(arg mesh_dir)"/>
   <!-- PiPER arm wrapper -->
@@ -518,4 +524,6 @@
     xyz="${arm_x} ${arm_y} ${arm_z}"
     rpy="0 0 0"
-    prefix="piper_"/>
+    prefix="piper_"
+    camera_xyz="${piper_camera_x} ${piper_camera_y} ${piper_camera_z}"
+    camera_rpy="${piper_camera_roll} ${piper_camera_pitch} ${piper_camera_yaw}"/>
 </robot>

Commit message: Refactor camera parameters in PiPER arm macros and update URDF files for consistency

File: src/ranger_description/urdf/piper_arm_macro.xacro (robot description, xacro)
@@ -4,6 +4,11 @@
   <xacro:include filename="$(find ranger_description)/urdf/piper_description_prefixed.xacro" />
   <!-- Wrapper macro to mount the PiPER arm to an arbitrary parent link. -->
-  <xacro:macro name="piper_arm" params="parent_link xyz:='0 0 0' rpy:='0 0 0' prefix:='piper_' camera_xyz:='0 0 0.05' camera_rpy:='0 0 0'">
-    <xacro:piper_with_gripper prefix="${prefix}" camera_xyz="${camera_xyz}" camera_rpy="${camera_rpy}" />
+  <xacro:macro name="piper_arm" params="parent_link xyz:='0 0 0' rpy:='0 0 0' prefix:='piper_' camera_xyz:='0 0 0.05' camera_roll:='0' camera_pitch:='0' camera_yaw:='0'">
+    <xacro:piper_with_gripper
+      prefix="${prefix}"
+      camera_xyz="${camera_xyz}"
+      camera_roll="${camera_roll}"
+      camera_pitch="${camera_pitch}"
+      camera_yaw="${camera_yaw}"/>
     <!--
       Mount PiPER's world link to the requested parent.

File: src/ranger_description/urdf/piper_description_prefixed.xacro (robot description, xacro)
@@ -14,5 +14,5 @@
     </transmission>
   </xacro:macro>
-  <xacro:macro name="piper_with_gripper" params="prefix:='piper_' camera_xyz:='0 0 0.05' camera_rpy:='0 0 0'">
+  <xacro:macro name="piper_with_gripper" params="prefix:='piper_' camera_xyz:='0 0 0.05' camera_roll:='0' camera_pitch:='0' camera_yaw:='0'">
   <!-- world -->
     <link name="${prefix}world"/>
@@ -405,12 +405,12 @@
         <origin xyz="0 0 0" rpy="0 0 0" />
         <mass value="0.07" />
-        <inertia ixx="0.00001298" ixy="0.0" ixz="0.0"
+        <inertia ixx="0.00001867" ixy="0.0" ixz="0.0"
                  iyy="0.00001298" iyz="0.0"
-                 izz="0.00001867" />
+                 izz="0.00001298" />
       </inertial>
       <visual>
         <origin xyz="0 0 0" rpy="0 0 0" />
         <geometry>
-          <box size="0.04 0.04 0.025"/>
+          <box size="0.025 0.04 0.04"/>
         </geometry>
         <material name="silver">
@@ -421,5 +421,5 @@
         <origin xyz="0 0 0" rpy="0 0 0" />
         <geometry>
-          <box size="0.04 0.04 0.025"/>
+          <box size="0.025 0.04 0.04"/>
         </geometry>
       </collision>
@@ -428,5 +428,5 @@
       <parent link="${prefix}gripper_base"/>
       <child link="${prefix}camera_link"/>
-      <origin xyz="${camera_xyz}" rpy="${camera_rpy}"/>
+      <origin xyz="${camera_xyz}" rpy="${camera_roll} ${camera_pitch - 1.5708} ${camera_yaw}"/>
     </joint>
     <link

File: src/ranger_description/urdf/ranger_complete.urdf.xacro (robot description, xacro)
@@ -16,7 +16,7 @@
   <xacro:property name="piper_camera_x" value="-0.085"/>
   <xacro:property name="piper_camera_y" value="0.0"/>
-  <xacro:property name="piper_camera_z" value="0.05"/>
+  <xacro:property name="piper_camera_z" value="0.04"/>
   <xacro:property name="piper_camera_roll" value="0.0"/>
-  <xacro:property name="piper_camera_pitch" value="0.5236"/>
+  <xacro:property name="piper_camera_pitch" value="0.0"/>
   <xacro:property name="piper_camera_yaw" value="0.0"/>
   <xacro:property name="mesh_dir" value="$(arg mesh_dir)"/>
@@ -526,4 +526,6 @@
     prefix="piper_"
     camera_xyz="${piper_camera_x} ${piper_camera_y} ${piper_camera_z}"
-    camera_rpy="${piper_camera_roll} ${piper_camera_pitch} ${piper_camera_yaw}"/>
+    camera_roll="${piper_camera_roll}"
+    camera_pitch="${piper_camera_pitch}"
+    camera_yaw="${piper_camera_yaw}"/>
 </robot>

Commit message: refactor: update end-effector link from piper_link6 to piper_tcp across multiple files

File: src/ranger_description/urdf/piper_arm_macro.xacro (robot description, xacro)
@@ -4,5 +4,5 @@
   <xacro:include filename="$(find ranger_description)/urdf/piper_description_prefixed.xacro" />
   <!-- Wrapper macro to mount the PiPER arm to an arbitrary parent link. -->
-  <xacro:macro name="piper_arm" params="parent_link xyz:='0 0 0' rpy:='0 0 0' prefix:='piper_' camera_xyz:='0 0 0.05' camera_roll:='0' camera_pitch:='0' camera_yaw:='0'">
+  <xacro:macro name="piper_arm" params="parent_link xyz:='0 0 0' rpy:='0 0 0' prefix:='piper_' camera_xyz:='0 0 0.05' camera_roll:='0' camera_pitch:='0' camera_yaw:='0' tcp_x:='0.0' tcp_y:='0.0' tcp_z:='0.14'">
     <xacro:piper_with_gripper
       prefix="${prefix}"
@@ -10,5 +10,8 @@
       camera_roll="${camera_roll}"
       camera_pitch="${camera_pitch}"
-      camera_yaw="${camera_yaw}"/>
+      camera_yaw="${camera_yaw}"
+      tcp_x="${tcp_x}"
+      tcp_y="${tcp_y}"
+      tcp_z="${tcp_z}"/>
     <!--
       Mount PiPER's world link to the requested parent.

File: src/ranger_description/urdf/piper_description_prefixed.xacro (robot description, xacro)
@@ -14,5 +14,5 @@
     </transmission>
   </xacro:macro>
-  <xacro:macro name="piper_with_gripper" params="prefix:='piper_' camera_xyz:='0 0 0.05' camera_roll:='0' camera_pitch:='0' camera_yaw:='0'">
+  <xacro:macro name="piper_with_gripper" params="prefix:='piper_' camera_xyz:='0 0 0.05' camera_roll:='0' camera_pitch:='0' camera_yaw:='0' tcp_x:='0.0' tcp_y:='0.0' tcp_z:='0.14'">
   <!-- world -->
     <link name="${prefix}world"/>
@@ -399,4 +399,10 @@
       <child
         link="${prefix}gripper_base" />
+    </joint>
+    <link name="${prefix}tcp"/>
+    <joint name="${prefix}joint6_to_tcp" type="fixed">
+      <origin xyz="${tcp_x} ${tcp_y} ${tcp_z}" rpy="0 0 0" />
+      <parent link="${prefix}link6" />
+      <child link="${prefix}tcp" />
     </joint>
     <!-- PiPER wrist camera (RealSense D405) -->

File: src/ranger_description/urdf/ranger_complete.urdf.xacro (robot description, xacro)
@@ -20,4 +20,7 @@
   <xacro:property name="piper_camera_pitch" value="0.3491"/>  <!-- 20 degrees -->
   <xacro:property name="piper_camera_yaw" value="0.0"/>
+  <xacro:property name="piper_tcp_x" value="0.0"/>
+  <xacro:property name="piper_tcp_y" value="0.0"/>
+  <xacro:property name="piper_tcp_z" value="0.14"/>
   <xacro:property name="mesh_dir" value="$(arg mesh_dir)"/>
   <!-- PiPER arm wrapper -->
@@ -528,4 +531,7 @@
     camera_roll="${piper_camera_roll}"
     camera_pitch="${piper_camera_pitch}"
-    camera_yaw="${piper_camera_yaw}"/>
+    camera_yaw="${piper_camera_yaw}"
+    tcp_x="${piper_tcp_x}"
+    tcp_y="${piper_tcp_y}"
+    tcp_z="${piper_tcp_z}"/>
 </robot>

Commit message: Add Ranger Mini 3.0 + PiPER arm simulation in Gazebo Fortress
- Created launch file to spawn the Ranger robot and start necessary controllers and bridges.
- Added URDF description for the Ranger robot with integrated sensors and controllers.
- Implemented a headless smoke test for the Gazebo simulation to verify core topics.
- Defined a garden world SDF for testing with various objects and obstacles.
- Included package.xml for ranger_sim with dependencies for simulation and control.
- Added .gitkeep file for models directory to maintain structure.

File: src/ranger_description/urdf/piper_arm_macro.xacro (robot description, xacro)
@@ -4,5 +4,5 @@
   <xacro:include filename="$(find ranger_description)/urdf/piper_description_prefixed.xacro" />
   <!-- Wrapper macro to mount the PiPER arm to an arbitrary parent link. -->
-  <xacro:macro name="piper_arm" params="parent_link xyz:='0 0 0' rpy:='0 0 0' prefix:='piper_' camera_xyz:='0 0 0.05' camera_roll:='0' camera_pitch:='0' camera_yaw:='0' tcp_x:='0.0' tcp_y:='0.0' tcp_z:='0.14'">
+  <xacro:macro name="piper_arm" params="parent_link xyz:='0 0 0' rpy:='0 0 0' prefix:='piper_' camera_xyz:='0 0 0.05' camera_roll:='0' camera_pitch:='0' camera_yaw:='0' tcp_x:='0.0' tcp_y:='0.0' tcp_z:='0.14' sim_gazebo_classic:='true'">
     <xacro:piper_with_gripper
       prefix="${prefix}"
@@ -13,5 +13,6 @@
       tcp_x="${tcp_x}"
       tcp_y="${tcp_y}"
-      tcp_z="${tcp_z}"/>
+      tcp_z="${tcp_z}"
+      sim_gazebo_classic="${sim_gazebo_classic}"/>
     <!--
       Mount PiPER's world link to the requested parent.

File: src/ranger_description/urdf/piper_description_prefixed.xacro (robot description, xacro)
@@ -14,5 +14,5 @@
     </transmission>
   </xacro:macro>
-  <xacro:macro name="piper_with_gripper" params="prefix:='piper_' camera_xyz:='0 0 0.05' camera_roll:='0' camera_pitch:='0' camera_yaw:='0' tcp_x:='0.0' tcp_y:='0.0' tcp_z:='0.14'">
+  <xacro:macro name="piper_with_gripper" params="prefix:='piper_' camera_xyz:='0 0 0.05' camera_roll:='0' camera_pitch:='0' camera_yaw:='0' tcp_x:='0.0' tcp_y:='0.0' tcp_z:='0.14' sim_gazebo_classic:='true'">
   <!-- world -->
     <link name="${prefix}world"/>
@@ -568,5 +568,6 @@
     <xacro:transmission_block tran_name="${prefix}tran7" joint_name="${prefix}joint7" motor_name="${prefix}motor7"/>
     <xacro:transmission_block tran_name="${prefix}tran8" joint_name="${prefix}joint8" motor_name="${prefix}motor8"/>
-  <!-- gazebo -->
+  <!-- Gazebo Classic ros2_control plugin (skipped when sim_gazebo_classic is false) -->
+    <xacro:if value="${sim_gazebo_classic}">
     <gazebo>
       <plugin name="gazebo_ros2_control" filename="libgazebo_ros2_control.so">
@@ -576,4 +577,5 @@
       </plugin>
     </gazebo>
+    </xacro:if>
     <!-- <gazebo reference="${prefix}base_link">
       <material>Gazebo/Black</material>

File: src/ranger_description/urdf/ranger_complete.urdf.xacro (robot description, xacro)
@@ -3,4 +3,6 @@
   <!-- Accept mesh directory as argument with default value -->
   <xacro:arg name="mesh_dir" default="package://ranger_description/meshes"/>
+  <!-- When false, the Gazebo Classic ros2_control plugin is omitted from the PiPER arm -->
+  <xacro:arg name="sim_gazebo_classic" default="true"/>
   <xacro:property name="M_PI" value="3.14159265359"/>
   <xacro:property name="base_to_footprint_z" value="0.33"/>
@@ -534,4 +536,5 @@
     tcp_x="${piper_tcp_x}"
     tcp_y="${piper_tcp_y}"
-    tcp_z="${piper_tcp_z}"/>
+    tcp_z="${piper_tcp_z}"
+    sim_gazebo_classic="$(arg sim_gazebo_classic)"/>
 </robot>
