Commit message: refactor: update mesh directory handling in PiPER arm and Gazebo launch files

File: src/ranger_description/urdf/piper_arm_macro.xacro (robot description, xacro)
@@ -4,5 +4,5 @@
   <xacro:include filename="$(find ranger_description)/urdf/piper_description_prefixed.xacro" />
   <!-- Wrapper macro to mount the PiPER arm to an arbitrary parent link. -->
-  <xacro:macro name="piper_arm" params="parent_link xyz:='0 0 0' rpy:='0 0 0' prefix:='piper_' camera_xyz:='0 0 0.05' camera_roll:='0' camera_pitch:='0' camera_yaw:='0' tcp_x:='0.0' tcp_y:='0.0' tcp_z:='0.14' sim_gazebo_classic:='true'">
+  <xacro:macro name="piper_arm" params="parent_link xyz:='0 0 0' rpy:='0 0 0' prefix:='piper_' camera_xyz:='0 0 0.05' camera_roll:='0' camera_pitch:='0' camera_yaw:='0' tcp_x:='0.0' tcp_y:='0.0' tcp_z:='0.14' sim_gazebo_classic:='true' mesh_dir:='package://piper_description/meshes'">
     <xacro:piper_with_gripper
       prefix="${prefix}"
@@ -14,5 +14,6 @@
       tcp_y="${tcp_y}"
       tcp_z="${tcp_z}"
-      sim_gazebo_classic="${sim_gazebo_classic}"/>
+      sim_gazebo_classic="${sim_gazebo_classic}"
+      mesh_dir="${mesh_dir}"/>
     <!--
       Mount PiPER's world link to the requested parent.

File: src/ranger_description/urdf/piper_description_prefixed.xacro (robot description, xacro)
@@ -14,5 +14,5 @@
     </transmission>
   </xacro:macro>
-  <xacro:macro name="piper_with_gripper" params="prefix:='piper_' camera_xyz:='0 0 0.05' camera_roll:='0' camera_pitch:='0' camera_yaw:='0' tcp_x:='0.0' tcp_y:='0.0' tcp_z:='0.14' sim_gazebo_classic:='true'">
+  <xacro:macro name="piper_with_gripper" params="prefix:='piper_' camera_xyz:='0 0 0.05' camera_roll:='0' camera_pitch:='0' camera_yaw:='0' tcp_x:='0.0' tcp_y:='0.0' tcp_z:='0.14' sim_gazebo_classic:='true' mesh_dir:='package://piper_description/meshes'">
   <!-- world -->
     <link name="${prefix}world"/>
@@ -35,19 +35,19 @@
         <geometry>
           <mesh
-            filename="package://piper_description/meshes/base_link.STL" />
-        </geometry>
-        <material
-          name="">
-          <color
-            rgba="0.792156862745098 0.819607843137255 0.933333333333333 1" />
-        </material>
-      </visual>
-      <collision>
-        <origin
-          xyz="0 0 0"
-          rpy="0 0 0" />
-        <geometry>
-          <mesh
-            filename="package://piper_description/meshes/base_link.STL" />
+            filename="${mesh_dir}/base_link.STL" />
+        </geometry>
+        <material
+          name="">
+          <color
+            rgba="0.792156862745098 0.819607843137255 0.933333333333333 1" />
+        </material>
+      </visual>
+      <collision>
+        <origin
+          xyz="0 0 0"
+          rpy="0 0 0" />
+        <geometry>
+          <mesh
+            filename="${mesh_dir}/base_link.STL" />
         </geometry>
       </collision>
@@ -66,19 +66,19 @@
         <geometry>
           <mesh
-            filename="package://piper_description/meshes/link1.STL" />
-        </geometry>
-        <material
-          name="">
-          <color
-            rgba="0.792156862745098 0.819607843137255 0.933333333333333 1" />
-        </material>
-      </visual>
-      <collision>
-        <origin
-          xyz="0 0 0"
-          rpy="0 0 0" />
-        <geometry>
-          <mesh
-            filename="package://piper_description/meshes/link1.STL" />
+            filename="${mesh_dir}/link1.STL" />
+        </geometry>
+        <material
+          name="">
+          <color
+            rgba="0.792156862745098 0.819607843137255 0.933333333333333 1" />
+        </material>
+      </visual>
+      <collision>
+        <origin
+          xyz="0 0 0"
+          rpy="0 0 0" />
+        <geometry>
+          <mesh
+            filename="${mesh_dir}/link1.STL" />
         </geometry>
       </collision>
@@ -115,19 +115,19 @@
         <geometry>
           <mesh
-            filename="package://piper_description/meshes/link2.STL" />
-        </geometry>
-        <material
-          name="">
-          <color
-            rgba="0.792156862745098 0.819607843137255 0.933333333333333 1" />
-        </material>
-      </visual>
-      <collision>
-        <origin
-          xyz="0 0 0"
-          rpy="0 0 0" />
-        <geometry>
-          <mesh
-            filename="package://piper_description/meshes/link2.STL" />
+            filename="${mesh_dir}/link2.STL" />
+        </geometry>
+        <material
+          name="">
+          <color
+            rgba="0.792156862745098 0.819607843137255 0.933333333333333 1" />
+        </material>
+      </visual>
+      <collision>
+        <origin
+          xyz="0 0 0"
+          rpy="0 0 0" />
+        <geometry>
+          <mesh
+            filename="${mesh_dir}/link2.STL" />
         </geometry>
       </collision>
@@ -165,19 +165,19 @@
         <geometry>
           <mesh
-            filename="package://piper_description/meshes/link3.STL" />
-        </geometry>
-        <material
-          name="">
-          <color
-            rgba="0.792156862745098 0.819607843137255 0.933333333333333 1" />
-        </material>
-      </visual>
-      <collision>
-        <origin
-          xyz="0 0 0"
-          rpy="0 0 0" />
-        <geometry>
-          <mesh
-            filename="package://piper_description/meshes/link3.STL" />
+            filename="${mesh_dir}/link3.STL" />
+        </geometry>
+        <material
+          name="">
+          <color
+            rgba="0.792156862745098 0.819607843137255 0.933333333333333 1" />
+        </material>
+      </visual>
+      <collision>
+        <origin
+          xyz="0 0 0"
+          rpy="0 0 0" />
+        <geometry>
+          <mesh
+            filename="${mesh_dir}/link3.STL" />
         </geometry>
       </collision>
@@ -215,19 +215,19 @@
         <geometry>
           <mesh
-            filename="package://piper_description/meshes/link4.STL" />
-        </geometry>
-        <material
-          name="">
-          <color
-            rgba="0.792156862745098 0.819607843137255 0.933333333333333 1" />
-        </material>
-      </visual>
-      <collision>
-        <origin
-          xyz="0 0 0"
-          rpy="0 0 0" />
-        <geometry>
-          <mesh
-            filename="package://piper_description/meshes/link4.STL" />
+            filename="${mesh_dir}/link4.STL" />
+        </geometry>
+        <material
+          name="">
+          <color
+            rgba="0.792156862745098 0.819607843137255 0.933333333333333 1" />
+        </material>
+      </visual>
+      <collision>
+        <origin
+          xyz="0 0 0"
+          rpy="0 0 0" />
+        <geometry>
+          <mesh
+            filename="${mesh_dir}/link4.STL" />
         </geometry>
       </collision>
@@ -264,19 +264,19 @@
         <geometry>
           <mesh
-            filename="package://piper_description/meshes/link5.STL" />
-        </geometry>
-        <material
-          name="">
-          <color
-            rgba="0.792156862745098 0.819607843137255 0.933333333333333 1" />
-        </material>
-      </visual>
-      <collision>
-        <origin
-          xyz="0 0 0"
-          rpy="0 0 0" />
-        <geometry>
-          <mesh
-            filename="package://piper_description/meshes/link5.STL" />
+            filename="${mesh_dir}/link5.STL" />
+        </geometry>
+        <material
+          name="">
+          <color
+            rgba="0.792156862745098 0.819607843137255 0.933333333333333 1" />
+        </material>
+      </visual>
+      <collision>
+        <origin
+          xyz="0 0 0"
+          rpy="0 0 0" />
+        <geometry>
+          <mesh
+            filename="${mesh_dir}/link5.STL" />
         </geometry>
       </collision>
@@ -313,5 +313,5 @@
         <geometry>
           <mesh
-            filename="package://piper_description/meshes/link6.STL" />
+            filename="${mesh_dir}/link6.STL" />
         </geometry>
         <material
@@ -327,5 +327,5 @@
         <geometry>
           <mesh
-            filename="package://piper_description/meshes/link6.STL" />
+            filename="${mesh_dir}/link6.STL" />
         </geometry>
       </collision>
@@ -371,19 +371,19 @@
         <geometry>
           <mesh
-            filename="package://piper_description/meshes/gripper_base.STL" />
-        </geometry>
-        <material
-          name="">
-          <color
-            rgba="0.792156862745098 0.819607843137255 0.933333333333333 1" />
-        </material>
-      </visual>
-      <collision>
-        <origin
-          xyz="0 0 0"
-          rpy="0 0 0" />
-        <geometry>
-          <mesh
-            filename="package://piper_description/meshes/gripper_base.STL" />
+            filename="${mesh_dir}/gripper_base.STL" />
+        </geometry>
+        <material
+          name="">
+          <color
+            rgba="0.792156862745098 0.819607843137255 0.933333333333333 1" />
+        </material>
+      </visual>
+      <collision>
+        <origin
+          xyz="0 0 0"
+          rpy="0 0 0" />
+        <geometry>
+          <mesh
+            filename="${mesh_dir}/gripper_base.STL" />
         </geometry>
       </collision>
@@ -465,19 +465,19 @@
         <geometry>
           <mesh
-            filename="package://piper_description/meshes/link7.STL" />
-        </geometry>
-        <material
-          name="">
-          <color
-            rgba="0.792156862745098 0.819607843137255 0.933333333333333 1" />
-        </material>
-      </visual>
-      <collision>
-        <origin
-          xyz="0 0 0"
-          rpy="0 0 0" />
-        <geometry>
-          <mesh
-            filename="package://piper_description/meshes/link7.STL" />
+            filename="${mesh_dir}/link7.STL" />
+        </geometry>
+        <material
+          name="">
+          <color
+            rgba="0.792156862745098 0.819607843137255 0.933333333333333 1" />
+        </material>
+      </visual>
+      <collision>
+        <origin
+          xyz="0 0 0"
+          rpy="0 0 0" />
+        <geometry>
+          <mesh
+            filename="${mesh_dir}/link7.STL" />
         </geometry>
       </collision>
@@ -523,19 +523,19 @@
         <geometry>
           <mesh
-            filename="package://piper_description/meshes/link8.STL" />
-        </geometry>
-        <material
-          name="">
-          <color
-            rgba="0.792156862745098 0.819607843137255 0.933333333333333 1" />
-        </material>
-      </visual>
-      <collision>
-        <origin
-          xyz="0 0 0"
-          rpy="0 0 0" />
-        <geometry>
-          <mesh
-            filename="package://piper_description/meshes/link8.STL" />
+            filename="${mesh_dir}/link8.STL" />
+        </geometry>
+        <material
+          name="">
+          <color
+            rgba="0.792156862745098 0.819607843137255 0.933333333333333 1" />
+        </material>
+      </visual>
+      <collision>
+        <origin
+          xyz="0 0 0"
+          rpy="0 0 0" />
+        <geometry>
+          <mesh
+            filename="${mesh_dir}/link8.STL" />
         </geometry>
       </collision>

File: src/ranger_description/urdf/piper_no_gripper_description_prefixed.xacro (robot description, xacro)
@@ -14,5 +14,5 @@
     </transmission>
   </xacro:macro>
-  <xacro:macro name="piper_no_gripper" params="prefix:='piper_'">
+  <xacro:macro name="piper_no_gripper" params="prefix:='piper_' mesh_dir:='package://piper_description/meshes'">
   <!-- world -->
     <link name="${prefix}world"/>
@@ -35,19 +35,19 @@
         <geometry>
           <mesh
-            filename="package://piper_description/meshes/base_link.STL" />
-        </geometry>
-        <material
-          name="">
-          <color
-            rgba="0.792156862745098 0.819607843137255 0.933333333333333 1" />
-        </material>
-      </visual>
-      <collision>
-        <origin
-          xyz="0 0 0"
-          rpy="0 0 0" />
-        <geometry>
-          <mesh
-            filename="package://piper_description/meshes/base_link.STL" />
+            filename="${mesh_dir}/base_link.STL" />
+        </geometry>
+        <material
+          name="">
+          <color
+            rgba="0.792156862745098 0.819607843137255 0.933333333333333 1" />
+        </material>
+      </visual>
+      <collision>
+        <origin
+          xyz="0 0 0"
+          rpy="0 0 0" />
+        <geometry>
+          <mesh
+            filename="${mesh_dir}/base_link.STL" />
         </geometry>
       </collision>
@@ -66,19 +66,19 @@
         <geometry>
           <mesh
-            filename="package://piper_description/meshes/link1.STL" />
-        </geometry>
-        <material
-          name="">
-          <color
-            rgba="0.792156862745098 0.819607843137255 0.933333333333333 1" />
-        </material>
-      </visual>
-      <collision>
-        <origin
-          xyz="0 0 0"
-          rpy="0 0 0" />
-        <geometry>
-          <mesh
-            filename="package://piper_description/meshes/link1.STL" />
+            filename="${mesh_dir}/link1.STL" />
+        </geometry>
+        <material
+          name="">
+          <color
+            rgba="0.792156862745098 0.819607843137255 0.933333333333333 1" />
+        </material>
+      </visual>
+      <collision>
+        <origin
+          xyz="0 0 0"
+          rpy="0 0 0" />
+        <geometry>
+          <mesh
+            filename="${mesh_dir}/link1.STL" />
         </geometry>
       </collision>
@@ -115,19 +115,19 @@
         <geometry>
           <mesh
-            filename="package://piper_description/meshes/link2.STL" />
-        </geometry>
-        <material
-          name="">
-          <color
-            rgba="0.792156862745098 0.819607843137255 0.933333333333333 1" />
-        </material>
-      </visual>
-      <collision>
-        <origin
-          xyz="0 0 0"
-          rpy="0 0 0" />
-        <geometry>
-          <mesh
-            filename="package://piper_description/meshes/link2.STL" />
+            filename="${mesh_dir}/link2.STL" />
+        </geometry>
+        <material
+          name="">
+          <color
+            rgba="0.792156862745098 0.819607843137255 0.933333333333333 1" />
+        </material>
+      </visual>
+      <collision>
+        <origin
+          xyz="0 0 0"
+          rpy="0 0 0" />
+        <geometry>
+          <mesh
+            filename="${mesh_dir}/link2.STL" />
         </geometry>
       </collision>
@@ -165,19 +165,19 @@
         <geometry>
           <mesh
-            filename="package://piper_description/meshes/link3.STL" />
-        </geometry>
-        <material
-          name="">
-          <color
-            rgba="0.792156862745098 0.819607843137255 0.933333333333333 1" />
-        </material>
-      </visual>
-      <collision>
-        <origin
-          xyz="0 0 0"
-          rpy="0 0 0" />
-        <geometry>
-          <mesh
-            filename="package://piper_description/meshes/link3.STL" />
+            filename="${mesh_dir}/link3.STL" />
+        </geometry>
+        <material
+          name="">
+          <color
+            rgba="0.792156862745098 0.819607843137255 0.933333333333333 1" />
+        </material>
+      </visual>
+      <collision>
+        <origin
+          xyz="0 0 0"
+          rpy="0 0 0" />
+        <geometry>
+          <mesh
+            filename="${mesh_dir}/link3.STL" />
         </geometry>
       </collision>
@@ -215,19 +215,19 @@
         <geometry>
           <mesh
-            filename="package://piper_description/meshes/link4.STL" />
-        </geometry>
-        <material
-          name="">
-          <color
-            rgba="0.792156862745098 0.819607843137255 0.933333333333333 1" />
-        </material>
-      </visual>
-      <collision>
-        <origin
-          xyz="0 0 0"
-          rpy="0 0 0" />
-        <geometry>
-          <mesh
-            filename="package://piper_description/meshes/link4.STL" />
+            filename="${mesh_dir}/link4.STL" />
+        </geometry>
+        <material
+          name="">
+          <color
+            rgba="0.792156862745098 0.819607843137255 0.933333333333333 1" />
+        </material>
+      </visual>
+      <collision>
+        <origin
+          xyz="0 0 0"
+          rpy="0 0 0" />
+        <geometry>
+          <mesh
+            filename="${mesh_dir}/link4.STL" />
         </geometry>
       </collision>
@@ -264,19 +264,19 @@
         <geometry>
           <mesh
-            filename="package://piper_description/meshes/link5.STL" />
-        </geometry>
-        <material
-          name="">
-          <color
-            rgba="0.792156862745098 0.819607843137255 0.933333333333333 1" />
-        </material>
-      </visual>
-      <collision>
-        <origin
-          xyz="0 0 0"
-          rpy="0 0 0" />
-        <geometry>
-          <mesh
-            filename="package://piper_description/meshes/link5.STL" />
+            filename="${mesh_dir}/link5.STL" />
+        </geometry>
+        <material
+          name="">
+          <color
+            rgba="0.792156862745098 0.819607843137255 0.933333333333333 1" />
+        </material>
+      </visual>
+      <collision>
+        <origin
+          xyz="0 0 0"
+          rpy="0 0 0" />
+        <geometry>
+          <mesh
+            filename="${mesh_dir}/link5.STL" />
         </geometry>
       </collision>
@@ -313,5 +313,5 @@
         <geometry>
           <mesh
-            filename="package://piper_description/meshes/link6.STL" />
+            filename="${mesh_dir}/link6.STL" />
         </geometry>
         <material
@@ -327,5 +327,5 @@
         <geometry>
           <mesh
-            filename="package://piper_description/meshes/link6.STL" />
+            filename="${mesh_dir}/link6.STL" />
         </geometry>
       </collision>

File: src/ranger_description/urdf/ranger_complete.urdf.xacro (robot description, xacro)
@@ -3,4 +3,5 @@
   <!-- Accept mesh directory as argument with default value -->
   <xacro:arg name="mesh_dir" default="package://ranger_description/meshes"/>
+  <xacro:arg name="piper_mesh_dir" default="package://piper_description/meshes"/>
   <!-- When false, the Gazebo Classic ros2_control plugin is omitted from the PiPER arm -->
   <xacro:arg name="sim_gazebo_classic" default="true"/>
@@ -537,4 +538,5 @@
     tcp_y="${piper_tcp_y}"
     tcp_z="${piper_tcp_z}"
-    sim_gazebo_classic="$(arg sim_gazebo_classic)"/>
+    sim_gazebo_classic="$(arg sim_gazebo_classic)"
+    mesh_dir="$(arg piper_mesh_dir)"/>
 </robot>

File: src/ranger_sim/urdf/ranger_gazebo.urdf.xacro (robot description, xacro)
@@ -4,5 +4,5 @@
   Includes the real robot description (with Gazebo Classic plugin disabled)
   and adds:
-    - Gazebo Fortress ros2_control plugin (ign_ros2_control) for the arm
+    - Gazebo Fortress ros2_control plugin (gz_ros2_control) for the arm
     - DiffDrive plugin for base mobility (holonomic approximation for v1)
     - Simulated Livox-style lidar
@@ -13,4 +13,5 @@
 <robot name="ranger_mini_complete" xmlns:xacro="http://ros.org/wiki/xacro">
   <xacro:arg name="mesh_dir" default="package://ranger_description/meshes"/>
+  <xacro:arg name="piper_mesh_dir" default="package://piper_description/meshes"/>
   <xacro:arg name="sim_gazebo_classic" default="false"/>
   <xacro:arg name="gz_controller_config" default="$(find ranger_sim)/config/ros2_controllers_sim.yaml"/>
@@ -24,5 +25,5 @@
   <ros2_control name="GazeboFortressSystem" type="system">
     <hardware>
-      <plugin>ign_ros2_control/IgnitionSystem</plugin>
+      <plugin>gz_ros2_control/GazeboSimSystem</plugin>
     </hardware>
     <!-- Arm joints 1-6 -->
@@ -71,6 +72,9 @@
   <!-- Gazebo Fortress system plugin to load the ros2_control hardware -->
   <gazebo>
-    <plugin filename="ign_ros2_control-system" name="ign_ros2_control::IgnitionROS2ControlPlugin">
+    <plugin filename="gz_ros2_control-system" name="gz_ros2_control::GazeboSimROS2ControlPlugin">
+      <robot_param>robot_description</robot_param>
+      <robot_param_node>robot_state_publisher</robot_param_node>
       <parameters>$(arg gz_controller_config)</parameters>
+      <controller_manager_name>controller_manager</controller_manager_name>
     </plugin>
   </gazebo>
