Commit message: update the ranger mini 3.0 urdf

File: src/ranger_description/urdf/ranger_complete.urdf.xacro (robot description, xacro)
@@ -1,14 +1,9 @@
-<?xml version="1.0"?>
-<robot xmlns:xacro="http://www.ros.org/wiki/xacro" name="ranger_mini_complete">
-  <!-- Constants -->
+<?xml version="1.0" encoding="utf-8"?>
+<robot name="ranger_mini_complete" xmlns:xacro="http://ros.org/wiki/xacro">
   <xacro:property name="M_PI" value="3.14159265359"/>
-  <!-- Base dimensions (Ranger Mini 3.0 approximate dimensions) -->
-  <xacro:property name="base_length" value="0.70"/>
-  <xacro:property name="base_width" value="0.70"/>
-  <xacro:property name="base_height" value="0.25"/>
-  <!-- Sensor mounting positions -->
-  <xacro:property name="lidar_x" value="0.0"/>
+  <xacro:property name="base_to_footprint_z" value="0.33"/>
+  <xacro:property name="lidar_x" value="0.33"/>
   <xacro:property name="lidar_y" value="0.0"/>
-  <xacro:property name="lidar_z" value="0.70"/>
+  <xacro:property name="lidar_z" value="0.0"/>
   <xacro:property name="camera_x" value="0.20"/>
   <xacro:property name="camera_y" value="0.0"/>
@@ -17,36 +12,430 @@
   <xacro:property name="arm_y" value="0.0"/>
   <xacro:property name="arm_z" value="0.30"/>
-  <!-- Base link -->
-  <link name="base_link">
-    <visual>
-      <geometry>
-        <box size="${base_length} ${base_width} ${base_height}"/>
-      </geometry>
-      <origin xyz="0 0 ${base_height/2}" rpy="0 0 0"/>
-      <material name="gray">
-        <color rgba="0.5 0.5 0.5 1.0"/>
-      </material>
-    </visual>
-    <collision>
-      <geometry>
-        <box size="${base_length} ${base_width} ${base_height}"/>
-      </geometry>
-      <origin xyz="0 0 ${base_height/2}" rpy="0 0 0"/>
-    </collision>
-    <inertial>
-      <mass value="50.0"/>
-      <origin xyz="0 0 ${base_height/2}" rpy="0 0 0"/>
-      <inertia ixx="2.042" ixy="0.0" ixz="0.0"
-               iyy="2.042" iyz="0.0"
-               izz="4.083"/>
-    </inertial>
-  </link>
-  <!-- Footprint link (for navigation) -->
+  <link
+    name="base_link">
+    <inertial>
+      <origin
+        xyz="-0.0242698272228022 -0.0030308024613212 0.0544267444673498"
+        rpy="0 0 0" />
+      <mass
+        value="10" />
+      <inertia ixx="0.1354" ixy="0.0" ixz="0.0" iyy="0.2417" iyz="0.0" izz="0.3085"/>
+    </inertial>
+    <visual>
+      <origin
+        xyz="0 0 0.0"
+        rpy="0 0 0" />
+      <geometry>
+        <mesh
+          filename="package://ranger_description/meshes/ranger_base.dae" scale="1000 1000 1000" />
+      </geometry>
+      <material
+        name="">
+        <color
+          rgba="0.792156862745098 0.819607843137255 0.933333333333333 1" />
+      </material>
+    </visual>
+        <collision>
+            <origin xyz="0 0 -0.1" rpy="0 0 0" />
+            <geometry>
+                <box size="0.5 0.35 0.2"/>
+            </geometry>
+        </collision>
+   </link>
   <link name="base_footprint"/>
   <joint name="base_footprint_joint" type="fixed">
     <parent link="base_footprint"/>
     <child link="base_link"/>
-    <origin xyz="0 0 0.10" rpy="0 0 0"/>
-  </joint>
+    <origin xyz="0 0 ${base_to_footprint_z}" rpy="0 0 0"/>
+  </joint>
+   <link
+    name="fr_steering_wheel_link">
+    <inertial>
+      <origin
+        xyz="1.8493E-05 1.2713E-06 0.043679"
+        rpy="0 0 0" />
+      <mass
+        value="1" />
+      <inertia
+        ixx="0.0063625"
+        ixy="-1.0581E-07"
+        ixz="-4.0831E-07"
+        iyy="0.006363"
+        iyz="-3.4944E-08"
+        izz="0.010465" />
+    </inertial>
+    <visual>
+      <origin
+        xyz="0 0 0"
+        rpy="0 0 0" />
+      <geometry>
+        <mesh filename="package://ranger_description/meshes/steering_wheel.dae" scale="10 10 10"/>
+      </geometry>
+      <material
+        name="">
+        <color
+          rgba="0.79216 0.81961 0.93333 1" />
+      </material>
+    </visual>
+    <collision>
+      <origin
+        xyz="0 0 0"
+        rpy="0 0 0" />
+      <geometry>
+          <cylinder radius="0.001" length="0.001"/>
+      </geometry>
+    </collision>
+  </link>
+  <joint
+    name="fr_steering_joint"
+    type="revolute">
+    <origin
+      xyz="0.25 -0.19 -0.1"
+      rpy="0 0 0" />
+    <parent
+      link="base_link" />
+    <child
+      link="fr_steering_wheel_link" />
+    <axis
+      xyz="0 0 -1" />
+    <limit effort="5" velocity="6.28"  lower="-2.1" upper="2.1" />
+  </joint>
+  <link name="fr_wheel_link">
+      <inertial>
+          <mass value="8" />
+          <origin xyz="0 0 0" />
+          <inertia ixx="0.02047" ixy="0.0" ixz="0.0" iyy="0.02047" iyz="0.0" izz="0.0324"/>
+          </inertial>
+      <visual>
+          <origin xyz="0 0 0" rpy="3.14 0 0" />
+          <geometry>
+            <mesh filename="package://ranger_description/meshes/wheel_v3.dae" scale="10 10 10"/>
+          </geometry>
+      </visual>
+      <collision>
+          <origin xyz="0 0 -0.005" rpy="1.57 0 0" />
+          <geometry>
+              <cylinder length="0.08" radius="0.09" />
+          </geometry>
+                <contact>
+                    <ode>
+                  <min_depth>0.001</min_depth>
+                    </ode>
+              </contact>
+      </collision>
+  </link>
+        <joint name="fr_wheel" type="continuous">
+            <origin xyz="0.0 0.0 -0.12" rpy="0 0 0" />
+            <parent link="fr_steering_wheel_link"/>
+            <child link="fr_wheel_link"/>
+            <axis xyz="0 1 0" rpy="0 0 0" />
+        </joint>
+  <link
+    name="fl_steering_wheel_link">
+    <inertial>
+      <origin
+        xyz="-0.0017956 -9.6304E-08 0.043642"
+        rpy="0 0 0" />
+      <mass
+        value="1" />
+      <inertia
+        ixx="0.0063695"
+        ixy="-2.1067E-08"
+        ixz="-0.00016867"
+        iyy="0.006363"
+        iyz="-1.0301E-08"
+        izz="0.010458" />
+    </inertial>
+    <visual>
+      <origin
+        xyz="0 0 0"
+        rpy="0 0 3.14" />
+      <geometry>
+        <mesh filename="package://ranger_description/meshes/steering_wheel.dae" scale="10 10 10"/>
+      </geometry>
+      <material
+        name="">
+        <color
+          rgba="0.79216 0.81961 0.93333 1" />
+      </material>
+    </visual>
+    <collision>
+      <origin
+        xyz="0 0 0"
+        rpy="0 0 0" />
+      <geometry>
+        <cylinder radius="0.001" length="0.001"/>
+      </geometry>
+    </collision>
+  </link>
+   <joint
+    name="fl_steering_joint"
+    type="revolute">
+    <origin
+      xyz="0.25 0.19 -0.1"
+      rpy="0 0 0" />
+    <parent
+      link="base_link" />
+    <child
+      link="fl_steering_wheel_link" />
+    <axis
+      xyz="0 0 -1" />
+        <limit effort="5" velocity="6.28"  lower="-2.1" upper="2.1" />
+  </joint>
+        <link name="fl_wheel_link">
+            <inertial>
+                <mass value="8" />
+                <origin xyz="0 0 0" />
+                <inertia ixx="0.02047" ixy="0.0" ixz="0.0" iyy="0.02047" iyz="0.0" izz="0.0324"/>
+            </inertial>
+            <visual>
+                <origin xyz="0 0 0" rpy="0 0 0" />
+                <geometry>
+                <mesh filename="package://ranger_description/meshes/wheel_v3.dae" scale="10 10 10"/>
+                </geometry>
+            </visual>
+            <collision>
+                <origin xyz="0 0 -0.005" rpy="1.57 0 0" />
+                <geometry>
+                    <cylinder length="0.08" radius="0.09" />
+                </geometry>
+                     <contact>
+                         <ode>
+                        <min_depth>0.001</min_depth>
+                         </ode>
+                    </contact>
+            </collision>
+        </link>
+        <joint name="fl_wheel" type="continuous">
+            <origin xyz="0.0 0.0 -0.12" rpy="0 0 0" />
+            <parent link="fl_steering_wheel_link"/>
+            <child link="fl_wheel_link"/>
+            <axis xyz="0 1 0" rpy="0 0 0" />
+        </joint>
+ <link
+    name="rl_steering_wheel_link">
+    <inertial>
+      <origin
+        xyz="-0.00017093 6.1255E-08 0.043678"
+        rpy="0 0 0" />
+      <mass
+        value="1" />
+      <inertia
+        ixx="0.0063627"
+        ixy="-2.1069E-08"
+        ixz="-1.587E-05"
+        iyy="0.006363"
+        iyz="9.3201E-09"
+        izz="0.010465" />
+    </inertial>
+    <visual>
+      <origin
+        xyz="0 0 0"
+        rpy="0 0 3.14" />
+      <geometry>
+        <mesh filename="package://ranger_description/meshes/steering_wheel.dae" scale="10 10 10"/>
+      </geometry>
+      <material
+        name="">
+        <color
+          rgba="0.79216 0.81961 0.93333 1" />
+      </material>
+    </visual>
+    <collision>
+      <origin
+        xyz="0 0 0"
+        rpy="0 0 0" />
+      <geometry>
+        <cylinder radius="0.001" length="0.001"/>
+      </geometry>
+    </collision>
+  </link>
+  <joint
+    name="rl_steering_joint"
+    type="revolute">
+    <origin
+      xyz="-0.25 0.19 -0.1"
+      rpy="0 0 0" />
+    <parent
+      link="base_link" />
+    <child
+      link="rl_steering_wheel_link" />
+    <axis
+      xyz="0 0 -1" />
+        <limit effort="5" velocity="6.28"  lower="-2.1" upper="2.1" />
+  </joint>
+        <link name="rl_wheel_link">
+            <inertial>
+                <mass value="8" />
+                <origin xyz="0 0 0" />
+                <inertia ixx="0.02047" ixy="0.0" ixz="0.0" iyy="0.02047" iyz="0.0" izz="0.0324"/>
+            </inertial>
+            <visual>
+                <origin xyz="0 0 0" rpy="0 0 0" />
+                <geometry>
+                  <mesh filename="package://ranger_description/meshes/wheel_v3.dae" scale="10 10 10"/>
+                </geometry>
+            </visual>
+            <collision>
+                <origin xyz="0.00 0.00 -0.005" rpy="1.57 0 0" />
+                <geometry>
+                    <cylinder length="0.08" radius="0.09" />
+                </geometry>
+                     <contact>
+                         <ode>
+                        <min_depth>0.001</min_depth>
+                         </ode>
+                    </contact>
+            </collision>
+        </link>
+        <joint name="rl_wheel" type="continuous">
+            <origin xyz="0.0 0.0 -0.12 " rpy="0 0 0" />
+            <parent link="rl_steering_wheel_link"/>
+            <child link="rl_wheel_link"/>
+            <axis xyz="0 1 0" rpy="0 0 0" />
+        </joint>
+   <link name="rr_steering_wheel_link">
+        <inertial>
+            <origin xyz="0.0 0.0 0.0"/>
+            <mass value="1"/>
+            <inertia ixx="0.01" ixy="0.0" ixz="0.0" iyy="0.01" iyz="0.0" izz="0.01"/>
+        </inertial>
+        <visual>
+          <origin
+            xyz="0 0 0"
+            rpy="0 0 0" />
+          <geometry>
+            <mesh filename="package://ranger_description/meshes/steering_wheel.dae" scale="10 10 10"/>
+          </geometry>
+        </visual>
+        <collision>
+            <origin  xyz="0 0 0" rpy="0 0 0" />
+                    <geometry>
+                <cylinder radius="0.001" length="0.001"/>
+            </geometry>
+        </collision>
+    </link>
+    <joint name="rr_steering_joint" type="revolute">
+        <origin xyz="-0.23 -0.206 -0.1" rpy="0 0 0" />
+        <parent link="base_link"/>
+        <child link="rr_steering_wheel_link"/>
+        <axis xyz="0 0 -1" rpy="0 0 0" />
+        <limit effort="5" velocity="6.28"  lower="-2.1" upper="2.1" />
+    </joint>
+       <link name="rr_wheel_link">
+            <inertial>
+                <mass value="8" />
+                <origin xyz="0 0 0" />
+                <inertia ixx="0.02047" ixy="0.0" ixz="0.0" iyy="0.02047" iyz="0.0" izz="0.0324"/>
+            </inertial>
+            <visual>
+                <origin xyz="0.0 0.0 0.0" rpy="3.14 0 0" />
+                <geometry>
+                    <mesh filename="package://ranger_description/meshes/wheel_v3.dae" scale="10 10 10"/>
+                </geometry>
+            </visual>
+            <collision>
+                <origin xyz="0.0 0.0 -0.005" rpy="1.57 0 0" />
+                <geometry>
+                    <cylinder length="0.08" radius="0.09" />
+                </geometry>
+                     <contact>
+                         <ode>
+                        <min_depth>0.001</min_depth>
+                         </ode>
+                    </contact>
+            </collision>
+        </link>
+        <joint name="rr_wheel" type="continuous">
+            <origin xyz="0.0 0.0 -0.12 " rpy="0 0 0" />
+            <parent link="rr_steering_wheel_link"/>
+            <child link="rr_wheel_link"/>
+            <axis xyz="0 1 0" rpy="0 0 0" />
+        </joint>
+<!--
+	<transmission name="fl_steering_wheel_trans">
+      <type>transmission_interface/SimpleTransmission</type>
+      <joint name="fl_steering_joint">
+		<hardwareInterface>hardware_interface/PositionJointInterface</hardwareInterface>
+      </joint>
+	  <actuator name="fl_steering_wheel_motor">
+		<hardwareInterface>hardware_interface/PositionJointInterface</hardwareInterface>
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
Commit message: Add launch task for Ranger complete bringup and update camera properties in URDF

File: src/ranger_description/urdf/ranger_complete.urdf.xacro (robot description, xacro)
@@ -6,7 +6,7 @@
   <xacro:property name="lidar_y" value="0.0"/>
   <xacro:property name="lidar_z" value="0.0"/>
-  <xacro:property name="camera_x" value="0.20"/>
+  <xacro:property name="camera_x" value="0.28"/>
   <xacro:property name="camera_y" value="0.0"/>
-  <xacro:property name="camera_z" value="0.50"/>
+  <xacro:property name="camera_z" value="0.115"/>
   <xacro:property name="arm_x" value="0.0"/>
   <xacro:property name="arm_y" value="0.0"/>
@@ -470,5 +470,5 @@
     <visual>
       <geometry>
-        <box size="0.090 0.025 0.025"/>
+        <box size="0.025 0.090 0.025"/>
       </geometry>
       <material name="silver">

Commit message: Update Ranger bringup launch and URDF to support mesh directory argument and add optional RViz visualization

File: src/ranger_description/urdf/ranger_complete.urdf.xacro (robot description, xacro)
@@ -1,4 +1,6 @@
 <?xml version="1.0" encoding="utf-8"?>
 <robot name="ranger_mini_complete" xmlns:xacro="http://ros.org/wiki/xacro">
+  <!-- Accept mesh directory as argument with default value -->
+  <xacro:arg name="mesh_dir" default="package://ranger_description/meshes"/>
   <xacro:property name="M_PI" value="3.14159265359"/>
   <xacro:property name="base_to_footprint_z" value="0.33"/>
@@ -12,4 +14,5 @@
   <xacro:property name="arm_y" value="0.0"/>
   <xacro:property name="arm_z" value="0.30"/>
+  <xacro:property name="mesh_dir" value="$(arg mesh_dir)"/>
   <link
     name="base_link">
@@ -28,5 +31,5 @@
       <geometry>
         <mesh
-          filename="package://ranger_description/meshes/ranger_base.dae" scale="1000 1000 1000" />
+          filename="${mesh_dir}/ranger_base.dae" scale="1000 1000 1000" />
       </geometry>
       <material
@@ -70,5 +73,5 @@
         rpy="0 0 0" />
       <geometry>
-        <mesh filename="package://ranger_description/meshes/steering_wheel.dae" scale="10 10 10"/>
+        <mesh filename="${mesh_dir}/steering_wheel.dae" scale="10 10 10"/>
       </geometry>
       <material
@@ -110,5 +113,5 @@
           <origin xyz="0 0 0" rpy="3.14 0 0" />
           <geometry>
-            <mesh filename="package://ranger_description/meshes/wheel_v3.dae" scale="10 10 10"/>
+            <mesh filename="${mesh_dir}/wheel_v3.dae" scale="10 10 10"/>
           </geometry>
       </visual>
@@ -152,5 +155,5 @@
         rpy="0 0 3.14" />
       <geometry>
-        <mesh filename="package://ranger_description/meshes/steering_wheel.dae" scale="10 10 10"/>
+        <mesh filename="${mesh_dir}/steering_wheel.dae" scale="10 10 10"/>
       </geometry>
       <material
@@ -192,5 +195,5 @@
                 <origin xyz="0 0 0" rpy="0 0 0" />
                 <geometry>
-                <mesh filename="package://ranger_description/meshes/wheel_v3.dae" scale="10 10 10"/>
+                <mesh filename="${mesh_dir}/wheel_v3.dae" scale="10 10 10"/>
                 </geometry>
             </visual>
@@ -234,5 +237,5 @@
         rpy="0 0 3.14" />
       <geometry>
-        <mesh filename="package://ranger_description/meshes/steering_wheel.dae" scale="10 10 10"/>
+        <mesh filename="${mesh_dir}/steering_wheel.dae" scale="10 10 10"/>
       </geometry>
       <material
@@ -274,5 +277,5 @@
                 <origin xyz="0 0 0" rpy="0 0 0" />
                 <geometry>
-                  <mesh filename="package://ranger_description/meshes/wheel_v3.dae" scale="10 10 10"/>
+                  <mesh filename="${mesh_dir}/wheel_v3.dae" scale="10 10 10"/>
                 </geometry>
             </visual>
@@ -306,5 +309,5 @@
             rpy="0 0 0" />
           <geometry>
-            <mesh filename="package://ranger_description/meshes/steering_wheel.dae" scale="10 10 10"/>
+            <mesh filename="${mesh_dir}/steering_wheel.dae" scale="10 10 10"/>
           </geometry>
         </visual>
@@ -332,5 +335,5 @@
                 <origin xyz="0.0 0.0 0.0" rpy="3.14 0 0" />
                 <geometry>
-                    <mesh filename="package://ranger_description/meshes/wheel_v3.dae" scale="10 10 10"/>
+                    <mesh filename="${mesh_dir}/wheel_v3.dae" scale="10 10 10"/>
                 </geometry>
             </visual>

Commit message: Add IMU frame and joint for LiDAR integration; update LiDAR link comment for clarity

File: src/ranger_description/urdf/ranger_complete.urdf.xacro (robot description, xacro)
@@ -441,5 +441,5 @@
     </plugin>
   </gazebo> -->
-  <!-- LiDAR Link (Livox Mid-360) -->
+  <!-- LiDAR Link (Livox Mid-360) - Physically mounted at 45° pitch -->
   <link name="lidar_link">
     <visual>
@@ -468,4 +468,11 @@
     <child link="lidar_link"/>
     <origin xyz="${lidar_x} ${lidar_y} ${lidar_z}" rpy="0 ${pi/4} 0"/>
+  </joint>
+  <!-- IMU frame inside LiDAR (for FASTLIO2) - aligned with lidar_link -->
+  <link name="imu_link"/>
+  <joint name="lidar_imu_joint" type="fixed">
+    <parent link="lidar_link"/>
+    <child link="imu_link"/>
+    <origin xyz="0 0 0" rpy="0 0 0"/>
   </joint>
   <!-- Camera Link (RealSense D435) -->

Commit message: Update documentation and configurations for Tier IV C2-176 camera integration

File: src/ranger_description/urdf/ranger_complete.urdf.xacro (robot description, xacro)
@@ -476,5 +476,5 @@
     <origin xyz="0 0 0" rpy="0 0 0"/>
   </joint>
-  <!-- Camera Link (RealSense D435) -->
+  <!-- Camera Link (Tier IV C2-176) -->
   <link name="camera_link">
     <visual>
@@ -504,16 +504,9 @@
     <origin xyz="${camera_x} ${camera_y} ${camera_z}" rpy="0 0 0"/>
   </joint>
-  <!-- Camera depth optical frame -->
-  <link name="camera_depth_optical_frame"/>
-  <joint name="camera_depth_optical_joint" type="fixed">
+  <!-- Camera optical frame -->
+  <link name="camera_optical_frame"/>
+  <joint name="camera_optical_joint" type="fixed">
     <parent link="camera_link"/>
-    <child link="camera_depth_optical_frame"/>
-    <origin xyz="0 0 0" rpy="${-M_PI/2} 0 ${-M_PI/2}"/>
-  </joint>
-  <!-- Camera color optical frame -->
-  <link name="camera_color_optical_frame"/>
-  <joint name="camera_color_optical_joint" type="fixed">
-    <parent link="camera_link"/>
-    <child link="camera_color_optical_frame"/>
+    <child link="camera_optical_frame"/>
     <origin xyz="0 0 0" rpy="${-M_PI/2} 0 ${-M_PI/2}"/>
   </joint>

Commit message: Add PiPER arm macros and update URDF files for integration

File: src/ranger_description/urdf/ranger_complete.urdf.xacro (robot description, xacro)
@@ -15,4 +15,6 @@
   <xacro:property name="arm_z" value="0.30"/>
   <xacro:property name="mesh_dir" value="$(arg mesh_dir)"/>
+  <!-- PiPER arm wrapper -->
+  <xacro:include filename="$(find ranger_description)/urdf/piper_arm_macro.xacro" />
   <link
     name="base_link">
@@ -511,31 +513,9 @@
     <origin xyz="0 0 0" rpy="${-M_PI/2} 0 ${-M_PI/2}"/>
   </joint>
-  <!-- PiPER Arm Base Link (placeholder - actual arm from piper_ros) -->
-  <link name="piper_base_link">
-    <visual>
-      <geometry>
-        <cylinder radius="0.06" length="0.10"/>
-      </geometry>
-      <material name="blue">
-        <color rgba="0.2 0.2 0.8 1.0"/>
-      </material>
-    </visual>
-    <collision>
-      <geometry>
-        <cylinder radius="0.06" length="0.10"/>
-      </geometry>
-    </collision>
-    <inertial>
-      <mass value="1.0"/>
-      <origin xyz="0 0 0"/>
-      <inertia ixx="0.01" ixy="0.0" ixz="0.0"
-               iyy="0.01" iyz="0.0"
-               izz="0.01"/>
-    </inertial>
-  </link>
-  <joint name="arm_mount" type="fixed">
-    <parent link="base_link"/>
-    <child link="piper_base_link"/>
-    <origin xyz="${arm_x} ${arm_y} ${arm_z}" rpy="0 0 0"/>
-  </joint>
+  <!-- PiPER arm -->
+  <xacro:piper_arm
+    parent_link="base_link"
+    xyz="${arm_x} ${arm_y} ${arm_z}"
+    rpy="0 0 0"
+    prefix="piper_"/>
 </robot>

Commit message: Update RViz launch detail and adjust PiPER arm properties in URDF

File: src/ranger_description/urdf/ranger_complete.urdf.xacro (robot description, xacro)
@@ -11,7 +11,7 @@
   <xacro:property name="camera_y" value="0.0"/>
   <xacro:property name="camera_z" value="0.115"/>
-  <xacro:property name="arm_x" value="0.0"/>
+  <xacro:property name="arm_x" value="0.15"/>
   <xacro:property name="arm_y" value="0.0"/>
-  <xacro:property name="arm_z" value="0.30"/>
+  <xacro:property name="arm_z" value="0.0"/>
   <xacro:property name="mesh_dir" value="$(arg mesh_dir)"/>
   <!-- PiPER arm wrapper -->

Commit message: Update PiPER camera pitch parameter to 15 degrees in ranger_complete.urdf.xacro

File: src/ranger_description/urdf/ranger_complete.urdf.xacro (robot description, xacro)
@@ -18,5 +18,5 @@
   <xacro:property name="piper_camera_z" value="0.04"/>
   <xacro:property name="piper_camera_roll" value="0.0"/>
-  <xacro:property name="piper_camera_pitch" value="0.0"/>
+  <xacro:property name="piper_camera_pitch" value="0.2618"/>  <!-- 15 degrees -->
   <xacro:property name="piper_camera_yaw" value="0.0"/>
   <xacro:property name="mesh_dir" value="$(arg mesh_dir)"/>

Commit message: update piper camera link to 20 degree

File: src/ranger_description/urdf/ranger_complete.urdf.xacro (robot description, xacro)
@@ -18,5 +18,5 @@
   <xacro:property name="piper_camera_z" value="0.04"/>
   <xacro:property name="piper_camera_roll" value="0.0"/>
-  <xacro:property name="piper_camera_pitch" value="0.2618"/>  <!-- 15 degrees -->
+  <xacro:property name="piper_camera_pitch" value="0.3491"/>  <!-- 20 degrees -->
   <xacro:property name="piper_camera_yaw" value="0.0"/>
   <xacro:property name="mesh_dir" value="$(arg mesh_dir)"/>
