Commit message: feat(calib): apply eye-in-hand camera mount calibration (wrist D405)
Wrist D405 camera mount (piper_camera_*) set from the converged eye-in-hand
calibration (MobileManipulationCore/config/handeye_calibration.yaml, spread 3.8mm):
x=-0.09455 y=0.00167 z=0.08620 roll=-0.10791 pitch=0.53414 yaw=0.11721. The grasp
XY is accurate on hardware with this mount (was nominal z=0.04 pitch=0.3491). The
residual fingertip-vs-tcp depth is handled by grasp_offset in the visual_servo node.

File: src/ranger_description/urdf/ranger_complete.urdf.xacro (robot description, xacro)
@@ -17,10 +17,14 @@
   <xacro:property name="arm_y" value="0.0"/>
   <xacro:property name="arm_z" value="0.077"/>
-  <xacro:property name="piper_camera_x" value="-0.085"/>
-  <xacro:property name="piper_camera_y" value="0.0"/>
-  <xacro:property name="piper_camera_z" value="0.04"/>
-  <xacro:property name="piper_camera_roll" value="0.0"/>
-  <xacro:property name="piper_camera_pitch" value="0.3491"/>  <!-- 20 degrees -->
-  <xacro:property name="piper_camera_yaw" value="0.0"/>
+  <!-- Wrist D405 mount from eye-in-hand calibration (handeye_orbit_calibrate.py,
+       MobileManipulationCore/config/handeye_calibration.yaml, spread 3.8mm).
+       XY verified correct on hardware; the grasp_offset_z handles the residual
+       fingertip depth. Nominal was x=-0.085 y=0 z=0.04 roll=0 pitch=0.3491 yaw=0. -->
+  <xacro:property name="piper_camera_x" value="-0.09455"/>
+  <xacro:property name="piper_camera_y" value="0.00167"/>
+  <xacro:property name="piper_camera_z" value="0.08620"/>
+  <xacro:property name="piper_camera_roll" value="-0.10791"/>
+  <xacro:property name="piper_camera_pitch" value="0.53414"/>
+  <xacro:property name="piper_camera_yaw" value="0.11721"/>
   <xacro:property name="piper_tcp_x" value="0.0"/>
   <xacro:property name="piper_tcp_y" value="0.0"/>
